Commit message: urdf tested

File: codebase/Beta/tests/ur5.urdf (robot description, URDF)
Before this commit: robot ur5, 0 links, 2 joints
Joints:
- added joint ee_joint: type fixed, parent link6, child ee_link, origin xyz=0 0.0823 0 rpy=-1.570796325 0 0, axis 0 0 1, limit lower=0 upper=0
- added joint joint2: type continuous, parent link1, child link2, origin xyz=0.0 0.13585 0.0 rpy=0.0 1.570796325 0.0, axis 0 1 0, limit lower=-3.14159 upper=3.14159
- added joint joint3: type continuous, parent link2, child link3, origin xyz=0.0 -0.1197 0.425 rpy=0.0 0.0 0.0, axis 0 1 0, limit lower=-3.14159 upper=3.14159
- added joint joint4: type continuous, parent link3, child link4, origin xyz=0.0 0.0 0.39225 rpy=0.0 1.570796325 0.0, axis 0 1 0, limit lower=-3.14159 upper=3.14159
- added joint joint5: type continuous, parent link4, child link5, origin xyz=0.0 0.093 0.0 rpy=0.0 0.0 0.0, axis 0 0 1, limit lower=-3.14159 upper=3.14159
- added joint joint6: type continuous, parent link5, child link6, origin xyz=0.0 0.0 0.09465 rpy=0.0 0.0 0.0, axis 0 1 0, limit lower=-3.14159 upper=3.14159
- joint joint1: limit (none) -> lower=-3.14159 upper=3.14159
- joint world_joint: limit (none) -> lower=0 upper=0
