Commit message: Tested main.cpp

File: codebase/Beta/tests/2_link.urdf (robot description, URDF)
Before this commit: robot 2_link_arm, 0 links, 4 joints
Joints:
- joint ee_joint: origin xyz=1 0 0 rpy=0 0 0 -> xyz=0.5 0 0 rpy=0 0 0
- joint joint1: limit lower=-3.14159 upper=3.14159 -> lower=-1.5707963268 upper=1.5707963268
